File: PCB Layouts/Motor Drivers/Motor Shield v2.0/motor_shield__SD_v2.0.brd (EAGLE design)
At the start: 77.1 x 52.1 mm, 26 parts

Commit message: Testing force control PID
Parts:
- removed MN1, MN2, MN3, MN4: (no value), sym:SOT23
- added Q1, Q2, Q3, Q4: MMBT2222A, SparkFun-DiscreteSemi:SOT23-3
- renumbered U$2 to C1
Connections:
- net *INHIBIT: now also Q4.1; no longer MN4.1
- net CURRENT_MONITOR: now also Q1.1; no longer MN1.1
- net CURRENT_REF: now also Q3.1; no longer MN2.1
- net DIRECTION: now also A1.15; no longer A1.30
- net FAULT_OUT: now also Q2.1; no longer MN3.1
- net GND: now also Q1.2, Q2.2, Q3.2, Q4.2; no longer MN1.2, MN2.2, MN3.2, MN4.2
- net N$15: now also Q1.3; no longer MN1.3
- net N$16: now also Q3.3; no longer MN2.3
- net N$30: now also Q2.3; no longer MN3.3
- net N$41: now also Q4.3; no longer MN4.3
- net PWM: now also A1.30; no longer A1.15
Routing:
- net DIRECTION: track 68.9 -> 57.1 mm
- net +5V: track 53.1 -> 61.2 mm
- net MOTOR_B: track 131.3 -> 133.8 mm
- net CURRENT_MONITOR: track 47.5 -> 48.2 mm

Commit message: Tiva shield
Connections:
- removed net N$51: A1.6
- net CURRENT_MONITOR: now also A1.6; no longer A1.38
Routing:
- net CURRENT_MONITOR: track 48.2 -> 57.8 mm, vias 1 -> 0
- net PWM: track 58.8 -> 60.4 mm
Other:
- board text added: "Motor Shield V2.0"
- board text removed: "Motor Shield V1.2"
Changed lines of the file:
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@@
 <wire x1="0" y1="52.06" x2="0" y2="0" width="0" layer="20"/>
 <text x="1.81" y="7.318" size="1.27" layer="21" rot="R180">1</text>
-<text x="74.338" y="3.194" size="1.778" layer="21" rot="R180">Motor Shield V1.2</text>
+<text x="74.338" y="3.194" size="1.778" layer="21" rot="R180">Motor Shield V2.0</text>
 <text x="10.84" y="45.09" size="1.778" layer="22" rot="MR180">Hall</text>
 </plain>
@@
 <contactref element="P1" pad="1"/>
 <contactref element="A1" pad="30"/>
-<wire x1="3.683" y1="6.35" x2="3.683" y2="3.817" width="0.4064" layer="1"/>
-<wire x1="3.683" y1="3.817" x2="6" y2="1.5" width="0.4064" layer="1"/>
-<wire x1="6" y1="1.5" x2="51.1" y2="1.5" width="0.4064" layer="1"/>
-<wire x1="51.1" y1="1.5" x2="53.5" y2="3.9" width="0.4064" layer="1"/>
-<wire x1="53.5" y1="3.9" x2="53.5" y2="4.8" width="0.4064" layer="1"/>
-<wire x1="53.5" y1="4.8" x2="51.6" y2="6.7" width="0.4064" layer="1"/>
-<wire x1="51.6" y1="6.7" x2="50.76" y2="6.7" width="0.4064" layer="1"/>
-<wire x1="50.76" y1="6.7" x2="50.7" y2="6.64" width="0.4064" layer="1"/>
+<wire x1="3.683" y1="6.35" x2="3.683" y2="3.417" width="0.4064" layer="1"/>
+<wire x1="3.683" y1="3.417" x2="6.3" y2="0.8" width="0.4064" layer="1"/>
+<wire x1="6.3" y1="0.8" x2="51.7" y2="0.8" width="0.4064" layer="1"/>
+<wire x1="51.7" y1="0.8" x2="53.4" y2="2.5" width="0.4064" layer="1"/>
+<wire x1="53.4" y1="2.5" x2="53.4" y2="5.2" width="0.4064" layer="1"/>
+<wire x1="53.4" y1="5.2" x2="52.3" y2="6.3" width="0.4064" layer="1"/>
+<wire x1="52.3" y1="6.3" x2="51.04" y2="6.3" width="0.4064" layer="1"/>
+<wire x1="51.04" y1="6.3" x2="50.7" y2="6.64" width="0.4064" layer="1"/>
 </signal>
 <signal name="GND">
@@
 <contactref element="P1" pad="4"/>
 <contactref element="R5" pad="2"/>
-<wire x1="3.937" y1="13.97" x2="3.937" y2="14.143" width="0.4064" layer="1"/>
+<wire x1="3.937" y1="14.143" x2="3.937" y2="13.97" width="0.4064" layer="1"/>
 <wire x1="8.414" y1="18.62" x2="3.937" y2="14.143" width="0.4064" layer="1"/>
-<via x="21.8" y="30.1" extent="1-16" drill="0.6" shape="square"/>
-<contactref element="A1" pad="38"/>
-<wire x1="21.8" y1="30.1" x2="23.5" y2="30.1" width="0.4064" layer="16"/>
-<wire x1="23.5" y1="30.1" x2="32.8" y2="39.4" width="0.4064" layer="16"/>
-<wire x1="32.8" y1="39.4" x2="32.8" y2="47.16" width="0.4064" layer="16"/>
-<wire x1="32.8" y1="47.16" x2="32.92" y2="47.28" width="0.4064" layer="16"/>
 <contactref element="Q1" pad="1"/>
 <wire x1="8.544" y1="18.75" x2="10.7" y2="18.75" width="0.4064" layer="1"/>
 <wire x1="8.544" y1="18.75" x2="8.414" y2="18.62" width="0.4064" layer="1"/>
-<wire x1="10.7" y1="18.75" x2="10.7" y2="20" width="0.4064" layer="1"/>
-<wire x1="10.7" y1="20" x2="20.8" y2="30.1" width="0.4064" layer="1"/>
-<wire x1="20.8" y1="30.1" x2="21.8" y2="30.1" width="0.4064" layer="1"/>
+<contactref element="A1" pad="6"/>
+<wire x1="3.937" y1="13.97" x2="5.53" y2="13.97" width="0.4064" layer="1"/>
+<wire x1="5.53" y1="13.97" x2="6.2" y2="13.3" width="0.4064" layer="1"/>
+<wire x1="6.2" y1="13.3" x2="6.2" y2="2.8" width="0.4064" layer="1"/>
+<wire x1="7.4" y1="1.6" x2="38.04" y2="1.6" width="0.4064" layer="1"/>
+<wire x1="38.04" y1="1.6" x2="40.54" y2="4.1" width="0.4064" layer="1"/>
+<wire x1="6.2" y1="2.8" x2="7.4" y2="1.6" width="0.4064" layer="1"/>
 </signal>
 <signal name="*INHIBIT">
@@
 <contactref element="A1" pad="5"/>
 </signal>
-<signal name="N$51">
-<contactref element="A1" pad="6"/>
-</signal>
 <signal name="N$52">
