File: PCB Layouts/Tiva boards/Shield v2.0/tm4cShield_v2.0.sch (EAGLE design)
At the start: 14 parts

Commit message: Tiva shield
Parts:
- removed ADC1, ADC3, ADC4: (no value), SparkFun-Connectors:CONN_02
- removed ENCODER: (no value), SparkFun-Connectors:CONN_03JST-PTH-VERT
- removed I2C: (no value), SparkFun-Connectors:I2C_STANDARD
- removed MOTOR: (no value), SparkFun-Connectors:CONN_04JST-PTH-VERT
- added ABSENC: x5, pel_molex:CONN_8-1-53261
- added C1, C3: 0.1uF, SparkFun-Capacitors:0.1UF-0603-25V-(+80/-20%)
- added C9: 2.2u, test_Beast_Elmo_Twitter_Carrier_Board_V1:2.2U_CAPACITOR_0603
- added D2: 12V, test_Beast_Elmo_Twitter_Carrier_Board_V1:YELLOW_LED_0603
- added D4: 5V, test_Beast_Elmo_Twitter_Carrier_Board_V1:BLUE_LED_0603
- added IC1: INA125U, burr-brown:INA125U
- added LOADCELL: x2, con-molex:53261-04
- added PS1: 12/5, murata-supplys:MURATA_NMG2405SC
- added R4: 1k, test_Beast_Elmo_Twitter_Carrier_Board_V1:1K_RESISTOR_0603
- added R5: 4k7, test_Beast_Elmo_Twitter_Carrier_Board_V1:4K7_RESISTOR_0603
- added R7, R8: 10k, SparkFun-Resistors:0.05OHM-0603-1/5W-1%
- added RG: 10k, SparkFun-Resistors:TRIMPOT-PTH-10MM-KNOB-1/2W-10%
- added THERMO: x4, con-molex:53261-03
- added TP3: GND, testpad:TP5000
- added TP4: 5V, testpad:TP5000
- added U$2: SN75175, RoMeLa:SN75175
- added U$4: SP490, RoMeLa:SP490
- added X1: x1, con-molex:53261-02
- added X11: (no value), pel_molex:CONN_10-1-53261
- ADC2: value (none) -> x3; device SparkFun-Connectors:CONN_02 -> con-molex:53261-02
Connections:
- net N$11 renamed PA5
- net N$12 renamed PA6
- net N$13 renamed PA7
- net N$18 renamed PD2
- net N$19 renamed PD3
- net N$30 renamed PC7
- net N$31 renamed PD6
- net N$32 renamed PD7
- net N$33 renamed PF4
- net N$37 renamed PF0
- net N$38 renamed RST
- net N$4 renamed PB0
- net N$42 renamed PA3
- net N$5 renamed PB1
- net N$8 renamed PE4
- net N$9 renamed PE5
- removed net N$22: A1.P$29
- removed net N$27: A1.P$37
- removed net N$28: A1.P$36
- removed net N$29: A1.P$35
- removed net N$36: A1.P$18
- removed net N$41: A1.P$13
- new net CASE: ABSENC.7
- new net CH_A: U$2.1A, X11.6
- new net CH_A*: U$2.1B, X11.5
- new net CH_B: U$2.2A, X11.8
- new net CH_B*: U$2.2B, X11.7
- new net CH_I: U$2.3A, X11.10
- new net CH_I*: U$2.3B, X11.9
- new net CLOCK+: ABSENC.2, U$4.Y
- new net CLOCK-: ABSENC.3, U$4.Z
- new net DATA+: ABSENC.4, U$4.A
- new net DATA-: ABSENC.5, U$4.B
- new net N$1: D4.A, R4.1
- new net N$10: IC1.RG@1, RG.WIPER
- new net N$14: A1.P$20
- new net N$17: U$2.4Y
- new net N$20: U$2.4A
- new net N$3: IC1.RG, RG.CCW
- new net N$35: D2.A, R5.1
- new net N$9: ABSENC.6
- new net PA4: A1.P$13, U$4.R
- new net PC4: A1.P$37, U$2.3Y
- new net PC5: A1.P$36, U$2.1Y
- new net PC6: A1.P$35, U$2.2Y
- new net PE0: A1.P$18, THERMO-2.S
- new net PE2: A1.P$28, ADC2-1.S
- new net PE3: A1.P$29, IC1.OUT, IC1.SENSE
- new net V+: LOADCELL-3.S
- new net V-: IC1.-IN, LOADCELL-2.S, R7.2
- new net VIN: C3.2, IC1.!SLEEP, IC1.+IN, IC1.V+, PS1.VIN+, R5.2, R8.1, X1-1.S
- new net V_2.5: IC1.REF, IC1.REF2.5, IC1.REFOUT, LOADCELL-4.S
- net 5V: now also ABSENC.1, C1.2, C9.1, PS1.VOUT+, R4.2, THERMO-1.S, TP4.TP, U$2.1,2EN, U$2.3,4EN, U$2.VCC, U$4.VCC, X11.2; no longer I2C.2, MOTOR.1
- net GND: now also ABSENC.8, ADC2-2.S, C1.1, C3.1, C9.2, D2.C, D4.C, IC1.REFCOM, IC1.V-, LOADCELL-1.S, PS1.VIN-, PS1.VOUT-, R7.1, R8.2, THERMO-3.S, TP3.TP, U$2.GND, U$4.GND, X1-2.S, X11.3; no longer A1.P$20, ADC1.2, ADC2.2, ADC3.2, ADC4.2, ENCODER.3, I2C.1, MOTOR.2, R1.1, R2.1, R3.1
- net N$21: now also U$2.4B; no longer A1.P$28
- net PA2: now also U$4.D; no longer MOTOR.4
- net PB2: no longer I2C.4
- net PB3: no longer I2C.3
- net PB4: no longer MOTOR.3
- net PB5: no longer ADC1.1
- net PB6: no longer ENCODER.1
- net PB7: no longer ENCODER.2
- net PD0: no longer ADC2.1
- net PD1: no longer ADC3.1
- net PE1: no longer ADC4.1
- net PF1: no longer LED1.A
- net PF2: no longer LED2.A
- net PF3: no longer LED3.A
Other:
- note added: "Abslute Encoder"
- note added: "Additional ADC"
- note added: "Connector"
- note added: "Direction PB7 PWM PF1 Current Sensor PE5"
- note added: "Encoder 0"
- note added: "Encoder 1"
- note added: "Encoder Conditioning"
- note added: "Incremental Encoder"
- note added: "Indication LED"
- note added: "Load Cell"
- note added: "Red 12V Green 5V"
- note added: "Test Point and protection"
- note added: "Thermocouple"
- note added: "Voltage Conversion"
- note removed: "ADC Input"
- note removed: "Encoder"
- note removed: "I2C"
