File: PCB Layouts/Tiva boards/SEA booster pack/tm4cShield_v2.0.brd (EAGLE design)
At the start: 51.7 x 64.8 mm, 42 parts, among them IC1 INA125U, U2 MCP2551, X1 x1

Commit message: RTOS clock
Parts:
- removed ADC1: x3, con-molex:53261-02
- removed LED1, LED2, LED3: (no value), EAGLE_BoosterPack_Library:LED-0603
- removed R3: (no value), EAGLE_BoosterPack_Library:RESC0603
- added BLUE, YELLOW: (no value), EAGLE_BoosterPack_Library:LED-0603
- added GPIO1: x7, con-molex:53261-02
- added GPIO2: x8, con-molex:53261-02
- added GPIO3: x9, con-molex:53261-02
- added SPI: x13, pel_molex:PB-53261-08
- added X10: I2C, con-molex:53261-04
- ADC2: value x3 -> x12
- THERMO: value x4 -> x3
- moved R2 39.9 mm to (43.7, 54.4)
- moved R1 39.3 mm to (43.7, 51.3)
- moved R6 3.30 mm to (38.4, 64.0), turned to 0 degrees
- moved D4 0.76 mm to (21.6, 52.1)
- moved R4 0.51 mm to (23.6, 52.1)
- moved X11 0.25 mm to (67.1, 70.4)
- renumbered U$2 to IC3, U$4 to IC2, U2 to IC4
Connections:
- removed net N$14: A1.20
- removed net N$15: ADC1.1
- removed net N$16: ADC1.2
- removed net N$7: LED3.C, R3.2
- new net N$36: SPI.3
- net 3.3V: now also SPI.1
- net 5V: now also SPI.8, THERMO.3, X10.1; no longer THERMO.1
- net GND: now also A1.20, GPIO1.2, GPIO2.2, GPIO3.2, R1.1, R2.1, SPI.2, THERMO.1, X10.4; no longer THERMO.3
- net N$2: now also BLUE.C; no longer LED1.C
- net N$6: now also YELLOW.C; no longer LED2.C
- net PA2: no longer IC2.3
- net PA5: now also IC2.3
- net PA6: now also X10.3
- net PA7: now also X10.2
- net PB6: now also GPIO1.1
- net PC7: now also YELLOW.A
- net PD3: now also SPI.4
- net PD7: now also BLUE.A
- net PE1: now also GPIO3.1
- net PF0: now also SPI.5
- net PF2: now also SPI.7
- net PF3: now also SPI.6
- net PF4: now also GPIO2.1
Routing:
- net 5V: track 46.2 -> 200.2 mm, vias 0 -> 6
- net GND: track 33.6 -> 127.6 mm, vias 0 -> 8
- net PD3: track 0.00 -> 70.7 mm
- net PA7: track 0.00 -> 70.4 mm
- net PA6: track 0.00 -> 66.4 mm
- net VIN: track 12.0 -> 72.7 mm, vias 0 -> 2
- net PF0: track 0.00 -> 48.3 mm
- net PF4: track 0.00 -> 47.3 mm
- net 3.3V: track 41.6 -> 80.2 mm, vias 2 -> 4
- net PA5: track 0.00 -> 37.1 mm, vias 0 -> 1
- net PF3: track 0.00 -> 36.8 mm
- net PD7: track 0.00 -> 32.3 mm
- net PC7: track 0.00 -> 31.8 mm
- net PF2: track 0.00 -> 30.8 mm
- net PE0: track 0.00 -> 24.3 mm
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- added copper zone on layer 1, net GND
- added copper zone on layer 16, net GND
Other:
- board text added: "IN"
- board text added: "INA125"
- board text added: "MCP"
- board text added: "S2"
- board text added: "SEA Shield"
- board text added: "SN75175"
- board text added: "v1.0"
- board text added: "x10"
- board text added: "x11"
- board text added: "x12"
- board text added: "x13"
- board text added: "x2"
- board text added: "x3"
- board text added: "x4"
- board text added: "x5"
- board text added: "x7"
- board text added: "x8"
- board text added: "x9"
