File: PCB Layouts/Tiva boards/SEA booster pack/tm4cShield_v2.0.sch (EAGLE design)
At the start: 42 parts, among them IC1 INA125U, U2 MCP2551, X1 x1

Commit message: RTOS clock
Parts:
- removed ADC1: x3, con-molex:53261-02
- removed LED1, LED2, LED3: (no value), EAGLE_BoosterPack_Library:LED0603
- removed R3: (no value), EAGLE_BoosterPack_Library:RESISTOR_0603
- added BLUE, YELLOW: (no value), EAGLE_BoosterPack_Library:LED0603
- added GPIO1: x7, con-molex:53261-02
- added GPIO2: x8, con-molex:53261-02
- added GPIO3: x9, con-molex:53261-02
- added SPI: x13, pel_molex:CONN_8-1-53261
- added X10: I2C, con-molex:53261-04
- ADC2: value x3 -> x12
- THERMO: value x4 -> x3
- renumbered U$2 to IC3, U$4 to IC2, U2 to IC4
Connections:
- removed net N$14: A1.P$20
- removed net N$15: ADC1-1.S
- removed net N$16: ADC1-2.S
- removed net N$7: LED3.C, R3.2
- new net N$36: SPI.3
- net 3.3V: now also SPI.1
- net 5V: now also SPI.8, THERMO-3.S, X10-1.S; no longer THERMO-1.S
- net GND: now also A1.P$20, GPIO1-2.S, GPIO2-2.S, GPIO3-2.S, R1.1, R2.1, SPI.2, THERMO-1.S, X10-4.S; no longer THERMO-3.S
- net N$2: now also BLUE.C; no longer LED1.C
- net N$6: now also YELLOW.C; no longer LED2.C
- net PA2: no longer IC2.D
- net PA5: now also IC2.D
- net PA6: now also X10-3.S
- net PA7: now also X10-2.S
- net PB6: now also GPIO1-1.S
- net PC7: now also YELLOW.A
- net PD3: now also SPI.4
- net PD7: now also BLUE.A
- net PE1: now also GPIO3-1.S
- net PF0: now also SPI.5
- net PF2: now also SPI.7
- net PF3: now also SPI.6
- net PF4: now also GPIO2-1.S
Other:
- note added: "Additional GPIO"
- note added: "Additional SPI"
- note added: "Debug LED"
- note added: "I2C"
- note added: "Reset"
- note added: "Tiva Connectors"
- note removed: "Connections"
- note removed: "Leds"
- moved on the sheet: ADC2-1, ADC2-2, C16, D2, D4, R13, R4, R5, S2, THERMO-1, THERMO-2, THERMO-3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
