File: PCB Layouts/Power Converter Boards/PowerCOnverter_v1.0.sch (EAGLE design)
At the start: 47 parts, among them Q1 PMBT3906, Q2 PMBT3906, Q3 PMBT3906, X1 48V, X2 12V, X3 24V, X4 15V

Commit message: MRAC adaptive control
Connections:
- removed net 15V: X4-1.S
- removed net 24V: PS3.+VIN
- net +15V: now also X4-1.S
- net +24V: now also PS3.+VIN
Changed lines of the file:
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@@
 <label x="279.4" y="101.6" size="1.778" layer="95" rot="R90"/>
+</segment>
+<segment>
+<pinref part="X4" gate="-1" pin="S"/>
+<wire x1="312.42" y1="165.1" x2="304.8" y2="165.1" width="0.1524" layer="91"/>
+<label x="304.8" y="165.1" size="1.778" layer="95" rot="R180" xref="yes"/>
 </segment>
 </net>
@@
 <pinref part="12" gate="G$1" pin="A"/>
 <wire x1="292.1" y1="81.28" x2="294.64" y2="81.28" width="0.1524" layer="91"/>
-</segment>
-</net>
-<net name="15V" class="0">
-<segment>
-<pinref part="X4" gate="-1" pin="S"/>
-<wire x1="312.42" y1="165.1" x2="304.8" y2="165.1" width="0.1524" layer="91"/>
-<label x="304.8" y="165.1" size="1.778" layer="95" rot="R180" xref="yes"/>
 </segment>
 </net>
@@
 </segment>
 </net>
-<net name="24V" class="0">
+<net name="+24V" class="0">
 <segment>
 <wire x1="78.74" y1="165.1" x2="91.44" y2="165.1" width="0.1524" layer="91"/>
